Commit message: Basic simulation with ros2 control and URDF

File: description/urdf/caddy_ai2.urdf.xacro (robot description, xacro)
@@ -3,5 +3,5 @@
   <!-- Import Caddy AI2 Materials macro -->
   <xacro:include filename="$(find caddy_ai2_ros2_gazebo_simulation)/description/urdf/materials.urdf.xacro" />
-  <xacro:macro name="caddy_ai2" params="parent prefix *origin is_simulation:=true">
+  <xacro:macro name="caddy_ai2" params="prefix *origin is_simulation:=true">
     <!-- Define tire properties - Deli Tire 18x8.5-8 (inches) -->
     <xacro:property name="wheel_radius" value="0.235"/>
@@ -31,9 +31,4 @@
     <!-- Base Link -->
     <link name="${prefix}base_link" />
-    <joint name="${prefix}world_joint" type="fixed">
-      <parent link="world"/>
-      <child link="${prefix}base_link"/>
-      <origin xyz="0 0 ${wheel_radius}" rpy="0 0 0"/>
-    </joint>
     <!-- Base Footprint -->
     <link name="${prefix}base_footprint"/>
@@ -75,5 +70,5 @@
     <!-- Rear Right Wheel -->
     <link name="${prefix}rear_right_wheel">
-      <collision>
+      <collision name="${prefix}rear_right_wheel_collision">
         <origin xyz="0 0 0" rpy="${PI/2} 0 ${PI/2}"/>
         <geometry>
@@ -105,5 +100,5 @@
     <!-- Rear Left Wheel -->
     <link name="${prefix}rear_left_wheel">
-        <collision>
+        <collision name="${prefix}rear_left_wheel_collision">
           <origin xyz="0 0 0" rpy="${PI/2} 0 ${PI/2}"/>
           <geometry>
@@ -167,6 +162,6 @@
     </joint>
     <!-- Front Right Wheel -->
-    <link name="front_right_wheel">
-      <collision>
+    <link name="${prefix}front_right_wheel">
+      <collision name="${prefix}front_right_wheel_collision">
         <geometry>
           <cylinder length="${wheel_width}" radius="${wheel_radius}"/>
@@ -196,5 +191,5 @@
     <!-- Front Left Wheel -->
     <link name="${prefix}front_left_wheel">
-      <collision>
+      <collision name="${prefix}front_left_wheel_collision">
         <geometry>
           <cylinder length="${wheel_width}" radius="${wheel_radius}"/>
@@ -256,6 +251,46 @@
       <gazebo>
         <plugin filename="gz_ros2_control-system" name="gz_ros2_control::GazeboSimROS2ControlPlugin">
-          <parameters>$(find caddy_ai2_ros2_gazebo_simulation)/bringup/config/simulation_controllers.yaml</parameters>
+          <parameters>$(find caddy_ai2_ros2_gazebo_simulation)/bringup/config/controllers_simulation.yaml</parameters>
         </plugin>
+      </gazebo>
+      <gazebo reference="${prefix}rear_right_wheel">
+        <plugin filename="gz-sim-contact-system" name="gz::sim::systems::Contact"/>
+        <sensor name="contact_sensor" type="contact">
+          <always_on>true</always_on>
+          <update_rate>1000</update_rate>
+          <contact>
+            <collision>${prefix}rear_right_wheel_collision</collision>
+          </contact>
+        </sensor>
+      </gazebo>
+      <gazebo reference="${prefix}rear_left_wheel">
+        <plugin filename="gz-sim-contact-system" name="gz::sim::systems::Contact"/>
+        <sensor name="contact_sensor" type="contact">
+          <always_on>true</always_on>
+          <update_rate>1000</update_rate>
+          <contact>
+            <collision>${prefix}rear_left_wheel_collision</collision>
+          </contact>
+        </sensor>
+      </gazebo>
+      <gazebo reference="${prefix}front_right_wheel">
+        <plugin filename="gz-sim-contact-system" name="gz::sim::systems::Contact"/>
+        <sensor name="contact_sensor" type="contact">
+          <always_on>true</always_on>
+          <update_rate>1000</update_rate>
+          <contact>
+            <collision>${prefix}front_right_wheel_collision</collision>
+          </contact>
+        </sensor>
+      </gazebo>
+      <gazebo reference="${prefix}front_left_wheel">
+        <plugin filename="gz-sim-contact-system" name="gz::sim::systems::Contact"/>
+        <sensor name="contact_sensor" type="contact">
+          <always_on>true</always_on>
+          <update_rate>1000</update_rate>
+          <contact>
+            <collision>${prefix}front_left_wheel_collision</collision>
+          </contact>
+        </sensor>
       </gazebo>
     </xacro:if>

File: description/urdf/sim_caddy_ai2.urdf.xacro (robot description, xacro)
@@ -4,10 +4,8 @@
   <xacro:arg name="prefix" default="" />
   <xacro:arg name="is_simulation" default="true" />
-  <!-- Used for fixing robot -->
-  <link name="world"/>
   <!-- Import Caddy AI2 description of the vehicle macro -->
   <xacro:include filename="$(find caddy_ai2_ros2_gazebo_simulation)/description/urdf/caddy_ai2.urdf.xacro" />
-  <xacro:caddy_ai2 parent="world" prefix="$(arg prefix)" is_simulation="$(arg is_simulation)">
-    <origin xyz="0 0 0" rpy="0 0 0" />
+  <xacro:caddy_ai2 prefix="$(arg prefix)" is_simulation="$(arg is_simulation)">
+    <origin xyz="0 0 0.235" rpy="0 0 0" />
   </xacro:caddy_ai2>
 </robot>
