Commit message: multispawn robots correcto

File: description/sdf/caddy_ai2_model.sdf.xacro (robot description, xacro)
@@ -1,189 +1,181 @@
 <?xml version="1.0" ?>
-<sdf version="1.11" xmlns:xacro="http://ros.org/wiki/xacro">
+<robot xmlns:xacro="http://ros.org/wiki/xacro">
   <!-- Include materials -->
   <xacro:include filename="$(find caddy_ai2_ros2_gazebo_simulation)/description/sdf/materials.sdf.xacro"/>
-  <!-- Define parameters with default values -->
-  <xacro:arg name="prefix" default="" />
-  <xacro:property name="prefix" value="$(arg prefix)" />
-  <model name='${prefix}caddy_ai2' canonical_link='${prefix}base_link'>
-    <!-- Define robot constants -->
-    <xacro:property name="wheel_radius" value="0.235"/>
-    <xacro:property name="wheel_width" value="0.22"/>
-    <xacro:property name="wheel_mass" value="8.7"/>
-    <xacro:property name="track_width" value="1"/>
-    <xacro:property name="wheelbase" value="1.65"/>
-    <xacro:property name="height" value="0.25"/>
-    <xacro:property name="mass" value="590"/>
-    <xacro:property name="inertial_origin_offset_x" value="-0.275"/>
-    <xacro:property name="inertial_origin_offset_z" value="${0.3-wheel_radius}"/>
-    <xacro:property name="max_steer_angle" value="0.5"/>
-    <xacro:property name="vehicle_collision_width" value="1.230"/>
-    <xacro:property name="vehicle_collision_length" value="2.660"/>
-    <xacro:property name="vehicle_collision_height" value="1.7"/>
-    <xacro:property name="vehicle_collision_offset_x" value="-0.25"/>
-    <xacro:property name="vehicle_collision_offset_z" value="${1.7/2 - wheel_radius}"/>
-    <xacro:property name="PI" value="3.1415926535897931"/>
-    <!-- Moments of inertia -->
-    <xacro:property name="rect_Ixx" value="${(1/12) * mass * (track_width**2 + height**2)}"/>
-    <xacro:property name="rect_Iyy" value="${(1/12) * mass * (wheelbase**2 + height**2)}"/>
-    <xacro:property name="rect_Izz" value="${(1/12) * mass * (wheelbase**2 + track_width**2)}"/>
-    <xacro:property name="wheel_Ixx" value="${(1/12) * wheel_mass * (3*wheel_radius**2 + wheel_width**2)}"/>
-    <xacro:property name="wheel_Iyy" value="${(1/12) * wheel_mass * (3*wheel_radius**2 + wheel_width**2)}"/>
-    <xacro:property name="wheel_Izz" value="${(1/2) * wheel_mass * wheel_radius**2}"/>
-    <!-- Initial Robot Pose -->
-    <pose> 0 0 ${wheel_radius} 0 0 0 </pose>
-    <!-- Robot Base -->
-    <link name='${prefix}base_link'>
-      <must_be_base_link>true</must_be_base_link>
-      <inertial>
-        <mass>${mass}</mass>
-        <pose>${inertial_origin_offset_x} 0 ${inertial_origin_offset_z} 0 0 0</pose>
-        <inertia>
-          <ixx>${rect_Ixx}</ixx><ixy>0</ixy><ixz>0</ixz>
-          <iyy>${rect_Iyy}</iyy><iyz>0</iyz><izz>${rect_Izz}</izz>
-        </inertia>
-      </inertial>
-      <visual name="${prefix}base_link_visual">
-        <geometry>
-          <mesh>
-            <uri>package://caddy_ai2_ros2_gazebo_simulation/description/meshes/stl/rbcar_chassis.stl</uri>
-          </mesh>
-        </geometry>
-        <xacro:material_color rgba="${color_white}"/>
-      </visual>
-      <collision name="${prefix}base_link_collision">
-        <pose>${vehicle_collision_offset_x} 0 ${vehicle_collision_offset_z} 0 0 0 </pose>
-        <geometry>
-          <box>
-            <size>${vehicle_collision_length} ${vehicle_collision_width} ${vehicle_collision_height}</size>
-          </box>
-        </geometry>
-      </collision>
-    </link>
-    <!-- Base Footprint -->
-    <link name="${prefix}base_footprint">
-      <pose relative_to="${prefix}base_link">${vehicle_collision_offset_x} 0.0 -${wheel_radius-0.01} 0 0 0</pose>
-      <visual name="${prefix}base_footprint_visual">
-        <geometry>
-          <box>
-            <size>${vehicle_collision_length} ${vehicle_collision_width} 0.01</size>
-          </box>
-        </geometry>
-        <xacro:material_color rgba="${color_red}"/>
-      </visual>
-    </link>
-    <joint name="${prefix}base_joint" type="fixed">
-      <parent>${prefix}base_link</parent>
-      <child>${prefix}base_footprint</child>
-      <pose relative_to='${prefix}base_footprint'/>
-    </joint>
-    <!-- === RUEDAS TRASERAS === -->
-    <xacro:macro name="rear_wheel" params="name suffix y_offset">
-      <link name="${prefix}${name}">
-        <pose relative_to="${prefix}base_link">-${wheelbase/2} ${y_offset} 0 0 0 ${PI/2}</pose>
-        <collision name="${prefix}${name}_collision">
-          <pose>0 0 0 ${PI/2} 0 ${PI/2}</pose>
+  <!-- ============================================ -->
+  <!-- MACRO PRINCIPAL DEL ROBOT                    -->
+  <!-- ============================================ -->
+  <xacro:macro name="caddy_ai2_robot" params="prefix:='' x:=0 y:=0 z:=0 yaw:=0">
+    <model name='${prefix}caddy_ai2' canonical_link='${prefix}base_link'>
+      <!-- === CONSTANTES DEL ROBOT === -->
+      <xacro:property name="wheel_radius" value="0.235"/>
+      <xacro:property name="wheel_width" value="0.22"/>
+      <xacro:property name="wheel_mass" value="8.7"/>
+      <xacro:property name="track_width" value="1"/>
+      <xacro:property name="wheelbase" value="1.65"/>
+      <xacro:property name="height" value="0.25"/>
+      <xacro:property name="mass" value="590"/>
+      <xacro:property name="inertial_origin_offset_x" value="-0.275"/>
+      <xacro:property name="inertial_origin_offset_z" value="${0.3-wheel_radius}"/>
+      <xacro:property name="max_steer_angle" value="0.5"/>
+      <xacro:property name="vehicle_collision_width" value="1.230"/>
+      <xacro:property name="vehicle_collision_length" value="2.660"/>
+      <xacro:property name="vehicle_collision_height" value="1.7"/>
+      <xacro:property name="vehicle_collision_offset_x" value="-0.25"/>
+      <xacro:property name="vehicle_collision_offset_z" value="${1.7/2 - wheel_radius}"/>
+      <xacro:property name="PI" value="3.1415926535897931"/>
+      <!-- Moments of inertia -->
+      <xacro:property name="rect_Ixx" value="${(1/12) * mass * (track_width**2 + height**2)}"/>
+      <xacro:property name="rect_Iyy" value="${(1/12) * mass * (wheelbase**2 + height**2)}"/>
+      <xacro:property name="rect_Izz" value="${(1/12) * mass * (wheelbase**2 + track_width**2)}"/>
+      <xacro:property name="wheel_Ixx" value="${(1/12) * wheel_mass * (3*wheel_radius**2 + wheel_width**2)}"/>
+      <xacro:property name="wheel_Iyy" value="${(1/12) * wheel_mass * (3*wheel_radius**2 + wheel_width**2)}"/>
+      <xacro:property name="wheel_Izz" value="${(1/2) * wheel_mass * wheel_radius**2}"/>
+      <!-- Pose inicial del robot (ahora parametrizada) -->
+      <pose>${x} ${y} ${z + wheel_radius} 0 0 ${yaw}</pose>
+      <!-- === LINKS Y JOINTS === -->
+      <!-- Robot Base -->
+      <link name='${prefix}base_link'>
+        <must_be_base_link>true</must_be_base_link>
+        <inertial>
+          <mass>${mass}</mass>
+          <pose>${inertial_origin_offset_x} 0 ${inertial_origin_offset_z} 0 0 0</pose>
+          <inertia>
+            <ixx>${rect_Ixx}</ixx><ixy>0</ixy><ixz>0</ixz>
+            <iyy>${rect_Iyy}</iyy><iyz>0</iyz><izz>${rect_Izz}</izz>
+          </inertia>
+        </inertial>
+        <visual name="${prefix}base_link_visual">
           <geometry>
-            <cylinder>
-              <length>${wheel_width}</length>
-              <radius>${wheel_radius}</radius>
-            </cylinder>
+            <mesh>
+              <uri>package://caddy_ai2_ros2_gazebo_simulation/description/meshes/stl/rbcar_chassis.stl</uri>
+            </mesh>
+          </geometry>
+          <xacro:material_color rgba="${color_white}"/>
+        </visual>
+        <collision name="${prefix}base_link_collision">
+          <pose>${vehicle_collision_offset_x} 0 ${vehicle_collision_offset_z} 0 0 0 </pose>
+          <geometry>
+            <box>
+              <size>${vehicle_collision_length} ${vehicle_collision_width} ${vehicle_collision_height}</size>
+            </box>
           </geometry>
         </collision>
-        <visual name="${prefix}${name}_visual">
-          <pose>0 0 0 ${PI/2} 0 ${PI/2}</pose>
+      </link>
+      <!-- Base Footprint -->
+      <link name="${prefix}base_footprint">
+        <pose relative_to="${prefix}base_link">${vehicle_collision_offset_x} 0.0 -${wheel_radius-0.01} 0 0 0</pose>
+        <visual name="${prefix}base_footprint_visual">
           <geometry>
-            <cylinder>
-              <length>${wheel_width}</length>
-              <radius>${wheel_radius}</radius>
-            </cylinder>
+            <box>
+              <size>${vehicle_collision_length} ${vehicle_collision_width} 0.01</size>
+            </box>
           </geometry>
-          <xacro:material_color rgba="${color_black}"/>
+          <xacro:material_color rgba="${color_red}"/>
         </visual>
-        <inertial>
-          <pose>0 0 0 ${PI/2} 0 ${PI/2}</pose>
-          <mass>${wheel_mass}</mass>
-          <inertia>
-            <ixx>${wheel_Ixx}</ixx><ixy>0</ixy><ixz>0</ixz>
-            <iyy>${wheel_Iyy}</iyy><iyz>0</iyz><izz>${wheel_Izz}</izz>
-          </inertia>
-        </inertial>
       </link>
-      <joint name="${prefix}${name}_joint" type="revolute">
+      <joint name="${prefix}base_joint" type="fixed">
         <parent>${prefix}base_link</parent>
-        <child>${prefix}${name}</child>
-        <pose relative_to='${prefix}${name}'/>
-        <axis>
-          <xyz expressed_in='__model__'>0 1 0</xyz>
-          <limit>
-            <lower>-1.79769e+308</lower>
-            <upper>1.79769e+308</upper>
-          </limit>
-        </axis>
+        <child>${prefix}base_footprint</child>
+        <pose relative_to='${prefix}base_footprint'/>
       </joint>
-    </xacro:macro>
-    <xacro:rear_wheel name="rear_right_wheel" suffix="rr" y_offset="-${track_width/2}"/>
-    <xacro:rear_wheel name="rear_left_wheel" suffix="rl" y_offset="${track_width/2}"/>
-    <!-- === RUEDAS DELANTERAS CON DIRECCIÓN === -->
-    <xacro:macro name="front_wheel_assembly" params="name y_offset steer_sign">
-      <!-- Steering link -->
-      <link name="${prefix}${name}_steer_link">
-        <pose relative_to="${prefix}base_link">${wheelbase/2} ${y_offset} 0 0 0 0</pose>
-      </link>
-      <joint name="${prefix}${name}_steer_joint" type="revolute">
-        <parent>${prefix}base_link</parent>
-        <child>${prefix}${name}_steer_link</child>
-        <pose relative_to='${prefix}${name}_steer_link'/>
-        <axis>
-          <xyz expressed_in='__model__'>0 0 1</xyz>
-          <limit>
-            <lower>${-max_steer_angle}</lower>
-            <upper>${max_steer_angle}</upper>
-          </limit>
-        </axis>
-      </joint>
-      <!-- Wheel link -->
-      <link name="${prefix}${name}">
-        <pose relative_to="${prefix}${name}_steer_link">0 0 0 -${PI/2} 0 0</pose>
-        <collision name="${prefix}${name}_collision">
-          <geometry>
-            <cylinder>
-              <length>${wheel_width}</length>
-              <radius>${wheel_radius}</radius>
-            </cylinder>
-          </geometry>
-        </collision>
-        <visual name="${prefix}${name}_visual">
-          <geometry>
-            <cylinder>
-              <length>${wheel_width}</length>
-              <radius>${wheel_radius}</radius>
-            </cylinder>
-          </geometry>
-          <xacro:material_color rgba="${color_black}"/>
-        </visual>
-        <inertial>
-          <mass>${wheel_mass}</mass>
-          <inertia>
-            <ixx>${wheel_Ixx}</ixx><ixy>0</ixy><ixz>0</ixz>
-            <iyy>${wheel_Iyy}</iyy><iyz>0</iyz><izz>${wheel_Izz}</izz>
-          </inertia>
-        </inertial>
-      </link>
-      <joint name="${prefix}${name}_joint" type="revolute">
-        <parent>${prefix}${name}_steer_link</parent>
-        <child>${prefix}${name}</child>
-        <pose relative_to="${prefix}${name}"/>
-        <axis>
-          <xyz expressed_in='__model__'>0 1 0</xyz>
-          <limit>
-            <lower>-1.79769e+308</lower>
-            <upper>1.79769e+308</upper>
-          </limit>
-        </axis>
-      </joint>
-    </xacro:macro>
-    <xacro:front_wheel_assembly name="front_right_wheel" y_offset="-${track_width/2}" steer_sign="1"/>
-    <xacro:front_wheel_assembly name="front_left_wheel" y_offset="${track_width/2}" steer_sign="1"/>
-  </model>
-</sdf>
+      <!-- === MACROS PARA RUEDAS === -->
+      <xacro:macro name="rear_wheel" params="name y_offset">
+        <link name="${prefix}${name}">
+          <pose relative_to="${prefix}base_link">-${wheelbase/2} ${y_offset} 0 0 0 ${PI/2}</pose>
+          <collision name="${prefix}${name}_collision">
+            <pose>0 0 0 ${PI/2} 0 ${PI/2}</pose>
+            <geometry>
+              <cylinder>
+                <length>${wheel_width}</length>
+                <radius>${wheel_radius}</radius>
+              </cylinder>
+            </geometry>
+          </collision>
+          <visual name="${prefix}${name}_visual">
+            <pose>0 0 0 ${PI/2} 0 ${PI/2}</pose>
+            <geometry>
+              <cylinder>
+                <length>${wheel_width}</length>
+                <radius>${wheel_radius}</radius>
+              </cylinder>
+            </geometry>
+            <xacro:material_color rgba="${color_black}"/>
+          </visual>
+          <inertial>
+            <pose>0 0 0 ${PI/2} 0 ${PI/2}</pose>
+            <mass>${wheel_mass}</mass>
+            <inertia>
+              <ixx>${wheel_Ixx}</ixx><ixy>0</ixy><ixz>0</ixz>
+              <iyy>${wheel_Iyy}</iyy><iyz>0</iyz><izz>${wheel_Izz}</izz>
+            </inertia>
+          </inertial>
+        </link>
+        <joint name="${prefix}${name}_joint" type="revolute">
+          <parent>${prefix}base_link</parent>
+          <child>${prefix}${name}</child>
+          <pose relative_to='${prefix}${name}'/>
+          <axis>
+            <xyz expressed_in='__model__'>0 1 0</xyz>
+            <limit><lower>-1e308</lower><upper>1e308</upper></limit>
+          </axis>
+        </joint>
+      </xacro:macro>
+      <xacro:macro name="front_wheel_assembly" params="name y_offset">
+        <link name="${prefix}${name}_steer_link">
+          <pose relative_to="${prefix}base_link">${wheelbase/2} ${y_offset} 0 0 0 0</pose>
+        </link>
+        <joint name="${prefix}${name}_steer_joint" type="revolute">
+          <parent>${prefix}base_link</parent>
+          <child>${prefix}${name}_steer_link</child>
+          <pose relative_to='${prefix}${name}_steer_link'/>
+          <axis>
+            <xyz expressed_in='__model__'>0 0 1</xyz>
+            <limit><lower>${-max_steer_angle}</lower><upper>${max_steer_angle}</upper></limit>
+          </axis>
+        </joint>
+        <link name="${prefix}${name}">
+          <pose relative_to="${prefix}${name}_steer_link">0 0 0 -${PI/2} 0 0</pose>
+          <collision name="${prefix}${name}_collision">
+            <geometry>
+              <cylinder>
+                <length>${wheel_width}</length>
+                <radius>${wheel_radius}</radius>
+              </cylinder>
+            </geometry>
+          </collision>
+          <visual name="${prefix}${name}_visual">
+            <geometry>
+              <cylinder>
+                <length>${wheel_width}</length>
+                <radius>${wheel_radius}</radius>
+              </cylinder>
+            </geometry>
+            <xacro:material_color rgba="${color_black}"/>
+          </visual>
+          <inertial>
+            <mass>${wheel_mass}</mass>
+            <inertia>
+              <ixx>${wheel_Ixx}</ixx><ixy>0</ixy><ixz>0</ixz>
+              <iyy>${wheel_Iyy}</iyy><iyz>0</iyz><izz>${wheel_Izz}</izz>
+            </inertia>
+          </inertial>
+        </link>
+        <joint name="${prefix}${name}_joint" type="revolute">
+          <parent>${prefix}${name}_steer_link</parent>
+          <child>${prefix}${name}</child>
+          <pose relative_to="${prefix}${name}"/>
+          <axis>
+            <xyz expressed_in='__model__'>0 1 0</xyz>
+            <limit><lower>-1e308</lower><upper>1e308</upper></limit>
+          </axis>
+        </joint>
+      </xacro:macro>
+      <!-- Instanciar ruedas -->
+      <xacro:rear_wheel name="rear_right_wheel" y_offset="-${track_width/2}"/>
+      <xacro:rear_wheel name="rear_left_wheel" y_offset="${track_width/2}"/>
+      <xacro:front_wheel_assembly name="front_right_wheel" y_offset="-${track_width/2}"/>
+      <xacro:front_wheel_assembly name="front_left_wheel" y_offset="${track_width/2}"/>
+    </model>
+  </xacro:macro>
+</robot>

File: description/sdf/caddy_ai2_world.sdf.xacro (robot description, xacro)
@@ -1,11 +1,31 @@
 <?xml version="1.0" ?>
 <sdf version="1.11" xmlns:xacro="http://ros.org/wiki/xacro">
-  <!-- Incluir materiales y el modelo del robot -->
+  <!-- SDF Specification 1.11 -->
+  <!-- https://sdformat.org/spec/1.11/sdf/ -->
+  <!-- ============================================ -->
+  <!-- 1. Definir argumentos globales               -->
+  <!-- ============================================ -->
+  <xacro:arg name="robot1_prefix" default="robot1_"/>
+  <xacro:arg name="robot1_x" default="0"/>
+  <xacro:arg name="robot1_y" default="0"/>
+  <xacro:arg name="robot1_yaw" default="0"/>
+  <xacro:arg name="robot2_prefix" default="robot2_"/>
+  <xacro:arg name="robot2_x" default="3"/>
+  <xacro:arg name="robot2_y" default="0"/>
+  <xacro:arg name="robot2_yaw" default="0"/>
+  <xacro:arg name="robot3_prefix" default="robot3_"/>
+  <xacro:arg name="robot3_x" default="-3"/>
+  <xacro:arg name="robot3_y" default="2"/>
+  <xacro:arg name="robot3_yaw" default="1.57"/>
+  <!-- ============================================ -->
+  <!-- 2. Incluir dependencias                      -->
+  <!-- ============================================ -->
   <xacro:include filename="$(find caddy_ai2_ros2_gazebo_simulation)/description/sdf/materials.sdf.xacro"/>
   <xacro:include filename="$(find caddy_ai2_ros2_gazebo_simulation)/description/sdf/caddy_ai2_model.sdf.xacro"/>
-  <!-- Parámetros del mundo -->
-  <xacro:arg name="prefix" default="" />
+  <!-- ============================================ -->
+  <!-- 3. Definir el mundo                          -->
+  <!-- ============================================ -->
   <world name='base_world'>
-    <!-- Configuración de física y plugins -->
+    <!-- Física y plugins (igual que antes) -->
     <physics name="1ms" type="ignored">
       <max_step_size>0.001</max_step_size>
@@ -19,5 +39,5 @@
       <render_engine>ogre2</render_engine>
     </plugin>
-    <!-- Iluminación -->
+    <!-- Luz solar -->
     <light name='sun' type='directional'>
       <cast_shadows>1</cast_shadows>
@@ -33,5 +53,5 @@
       <direction>-0.5 0.1 -0.9</direction>
     </light>
-    <!-- Plano de suelo -->
+    <!-- Ground plane -->
     <model name='ground_plane'>
       <static>1</static>
@@ -98,9 +118,32 @@
       </camera>
     </gui>
-    <!-- === INCLUSIÓN DEL MODELO DEL ROBOT === -->
-    <!-- Pose inicial del robot en el mundo -->
-    <xacro:caddy_ai2_model prefix="$(arg prefix)"/>
-    <!-- Nota: si no usas macro wrapper, simplemente copia el contenido del modelo aquí
-         o usa <include> si conviertes el modelo a SDF puro -->
+    <!-- ============================================ -->
+    <!-- 4. Instanciar múltiples robots               -->
+    <!-- ============================================ -->
+    <!-- Robot 1 -->
+    <xacro:caddy_ai2_robot
+      prefix=""
+      x="0"
+      y="0"
+      yaw="180"/>
+    <!--<xacro:caddy_ai2_robot
+      prefix="$(arg robot1_prefix)"
+      x="$(arg robot1_x)"
+      y="$(arg robot1_y)"
+      yaw="$(arg robot1_yaw)"/>-->
+    <!-- Robot 2 -->
+    <!--<xacro:caddy_ai2_robot
+      prefix="$(arg robot2_prefix)"
+      x="$(arg robot2_x)"
+      y="$(arg robot2_y)"
+      yaw="$(arg robot2_yaw)"/>-->
+    <!-- Robot 3 (descomentar si se necesita) -->
+    <!--
+    <xacro:caddy_ai2_robot
+      prefix="$(arg robot3_prefix)"
+      x="$(arg robot3_x)"
+      y="$(arg robot3_y)"
+      yaw="$(arg robot3_yaw)"/>
+    -->
   </world>
 </sdf>
