Commit message: Simulación ante desarrollo

File: description/sdf/caddy_ai2_model.sdf.xacro (robot description, xacro)
@@ -32,8 +32,7 @@
       <xacro:property name="wheel_Iyy" value="${(1/12) * wheel_mass * (3*wheel_radius**2 + wheel_width**2)}"/>
       <xacro:property name="wheel_Izz" value="${(1/2) * wheel_mass * wheel_radius**2}"/>
-      <!-- Pose inicial del robot (ahora parametrizada) -->
+      <!-- Pose inicial parametrizada -->
       <pose>${x} ${y} ${z + wheel_radius} 0 0 ${yaw}</pose>
-      <!-- === LINKS Y JOINTS === -->
-      <!-- Robot Base -->
+      <!-- ==================== ROBOT BASE ==================== -->
       <link name='${prefix}base_link'>
         <must_be_base_link>true</must_be_base_link>
@@ -80,5 +79,6 @@
         <pose relative_to='${prefix}base_footprint'/>
       </joint>
-      <!-- === MACROS PARA RUEDAS === -->
+      <!-- ==================== MACROS PARA RUEDAS ==================== -->
+      <!-- Ruedas traseras: control de VELOCIDAD -->
       <xacro:macro name="rear_wheel" params="name y_offset">
         <link name="${prefix}${name}">
@@ -119,8 +119,20 @@
             <xyz expressed_in='__model__'>0 1 0</xyz>
             <limit><lower>-1e308</lower><upper>1e308</upper></limit>
+            <dynamics damping="0.01" friction="0.01"/>
           </axis>
+          <!-- === gz_ros2_control: VELOCITY para tracción === -->
+          <gz_ros2_control>
+            <command_interface name="velocity">
+              <param name="min">-10</param>
+              <param name="max">10</param>
+            </command_interface>
+            <state_interface name="velocity"/>
+            <state_interface name="position"/>
+          </gz_ros2_control>
         </joint>
       </xacro:macro>
+      <!-- Ruedas delanteras: steering con control de POSICIÓN + wheel pasivo -->
       <xacro:macro name="front_wheel_assembly" params="name y_offset">
+        <!-- Steering joint: control de POSICIÓN -->
         <link name="${prefix}${name}_steer_link">
           <pose relative_to="${prefix}base_link">${wheelbase/2} ${y_offset} 0 0 0 0</pose>
@@ -133,6 +145,16 @@
             <xyz expressed_in='__model__'>0 0 1</xyz>
             <limit><lower>${-max_steer_angle}</lower><upper>${max_steer_angle}</upper></limit>
+            <dynamics damping="1.0" friction="0.1"/>
           </axis>
+          <!-- === gz_ros2_control: POSITION para dirección === -->
+          <gz_ros2_control>
+            <command_interface name="position">
+              <param name="min">-${max_steer_angle}</param>
+              <param name="max">${max_steer_angle}</param>
+            </command_interface>
+            <state_interface name="position"/>
+          </gz_ros2_control>
         </joint>
+        <!-- Wheel joint: solo estado (sigue pasivamente al steering) -->
         <link name="${prefix}${name}">
           <pose relative_to="${prefix}${name}_steer_link">0 0 0 -${PI/2} 0 0</pose>
@@ -170,7 +192,12 @@
             <limit><lower>-1e308</lower><upper>1e308</upper></limit>
           </axis>
+          <!-- === Solo state interfaces para rueda delantera === -->
+          <gz_ros2_control>
+            <state_interface name="position"/>
+            <state_interface name="velocity"/>
+          </gz_ros2_control>
         </joint>
       </xacro:macro>
-      <!-- Instanciar ruedas -->
+      <!-- ==================== INSTANCIAR RUEDAS ==================== -->
       <xacro:rear_wheel name="rear_right_wheel" y_offset="-${track_width/2}"/>
       <xacro:rear_wheel name="rear_left_wheel" y_offset="${track_width/2}"/>

File: description/sdf/caddy_ai2_world.sdf.xacro (robot description, xacro)
@@ -126,5 +126,5 @@
       x="0"
       y="0"
-      yaw="180"/>
+      yaw="0"/>
     <!--<xacro:caddy_ai2_robot
       prefix="$(arg robot1_prefix)"

Commit message: Simulation

File: description/sdf/caddy_ai2_model.sdf.xacro (robot description, xacro)
@@ -1,4 +1,51 @@
 <?xml version="1.0" ?>
 <sdf version="1.11" xmlns:xacro="http://ros.org/wiki/xacro">
+  <!-- ============================================ -->
+  <!-- Arguments (overridable from CLI or launch)   -->
+  <!-- ============================================ -->
+  <xacro:arg name="prefix"          default=""/>
+  <xacro:arg name="namespace"       default=""/>
+  <xacro:arg name="wheelbase"       default="1.65"/>
+  <xacro:arg name="track_width"     default="1.0"/>
+  <xacro:arg name="wheel_radius"    default="0.235"/>
+  <xacro:arg name="max_steer_angle" default="0.4"/>
+  <xacro:arg name="wheel_width"                default="0.22"/>
+  <xacro:arg name="wheel_mass"                 default="8.7"/>
+  <xacro:arg name="height"                     default="0.25"/>
+  <xacro:arg name="mass"                       default="590"/>
+  <xacro:arg name="vehicle_collision_width"    default="1.230"/>
+  <xacro:arg name="vehicle_collision_length"   default="2.660"/>
+  <xacro:arg name="vehicle_collision_height"   default="1.7"/>
+  <xacro:arg name="vehicle_collision_offset_x" default="-0.25"/>
+  <xacro:arg name="inertial_origin_offset_x"   default="-0.275"/>
+  <!-- ============================================ -->
+  <!-- Robot constants                              -->
+  <!-- ============================================ -->
+  <!-- Parameterizable (from robot_params.yaml via launch) -->
+  <xacro:property name="wheelbase"       value="$(arg wheelbase)"/>
+  <xacro:property name="track_width"     value="$(arg track_width)"/>
+  <xacro:property name="wheel_radius"    value="$(arg wheel_radius)"/>
+  <xacro:property name="max_steer_angle" value="$(arg max_steer_angle)"/>
+  <!-- Fixed structural properties -->
+  <xacro:property name="wheel_width"                value="$(arg wheel_width)"/>
+  <xacro:property name="wheel_mass"                 value="$(arg wheel_mass)"/>
+  <xacro:property name="height"                     value="$(arg height)"/>
+  <xacro:property name="mass"                       value="$(arg mass)"/>
+  <xacro:property name="PI"                         value="3.1415926535897931"/>
+  <xacro:property name="vehicle_collision_width"    value="$(arg vehicle_collision_width)"/>
+  <xacro:property name="vehicle_collision_length"   value="$(arg vehicle_collision_length)"/>
+  <xacro:property name="vehicle_collision_height"   value="$(arg vehicle_collision_height)"/>
+  <xacro:property name="vehicle_collision_offset_x" value="$(arg vehicle_collision_offset_x)"/>
+  <xacro:property name="inertial_origin_offset_x"   value="$(arg inertial_origin_offset_x)"/>
+  <!-- Derived geometry -->
+  <xacro:property name="inertial_origin_offset_z"   value="${0.3 - wheel_radius}"/>
+  <xacro:property name="vehicle_collision_offset_z" value="${vehicle_collision_height / 2 - wheel_radius}"/>
+  <!-- Moments of inertia -->
+  <xacro:property name="rect_Ixx"  value="${(1/12) * mass * (track_width**2 + height**2)}"/>
+  <xacro:property name="rect_Iyy"  value="${(1/12) * mass * (wheelbase**2 + height**2)}"/>
+  <xacro:property name="rect_Izz"  value="${(1/12) * mass * (wheelbase**2 + track_width**2)}"/>
+  <xacro:property name="wheel_Ixx" value="${(1/12) * wheel_mass * (3*wheel_radius**2 + wheel_width**2)}"/>
+  <xacro:property name="wheel_Iyy" value="${(1/12) * wheel_mass * (3*wheel_radius**2 + wheel_width**2)}"/>
+  <xacro:property name="wheel_Izz" value="${(1/2) * wheel_mass * wheel_radius**2}"/>
   <!-- Include materials -->
   <xacro:include filename="$(find caddy_ai2_ros2_gazebo_simulation)/description/sdf/materials.sdf.xacro"/>
@@ -7,32 +54,25 @@
   <!-- ============================================ -->
   <xacro:macro name="caddy_ai2_robot" params="prefix:='' namespace:=''">
-    <model name='${prefix}caddy_ai2' canonical_link='${prefix}base_link'>
-      <!-- === CONSTANTES DEL ROBOT === -->
-      <xacro:property name="wheel_radius" value="0.235"/>
-      <xacro:property name="wheel_width" value="0.22"/>
-      <xacro:property name="wheel_mass" value="8.7"/>
-      <xacro:property name="track_width" value="1"/>
-      <xacro:property name="wheelbase" value="1.65"/>
-      <xacro:property name="height" value="0.25"/>
-      <xacro:property name="mass" value="590"/>
-      <xacro:property name="inertial_origin_offset_x" value="-0.275"/>
-      <xacro:property name="inertial_origin_offset_z" value="${0.3-wheel_radius}"/>
-      <xacro:property name="max_steer_angle" value="0.5"/>
-      <xacro:property name="vehicle_collision_width" value="1.230"/>
-      <xacro:property name="vehicle_collision_length" value="2.660"/>
-      <xacro:property name="vehicle_collision_height" value="1.7"/>
-      <xacro:property name="vehicle_collision_offset_x" value="-0.25"/>
-      <xacro:property name="vehicle_collision_offset_z" value="${1.7/2 - wheel_radius}"/>
-      <xacro:property name="PI" value="3.1415926535897931"/>
-      <!-- Moments of inertia -->
-      <xacro:property name="rect_Ixx" value="${(1/12) * mass * (track_width**2 + height**2)}"/>
-      <xacro:property name="rect_Iyy" value="${(1/12) * mass * (wheelbase**2 + height**2)}"/>
-      <xacro:property name="rect_Izz" value="${(1/12) * mass * (wheelbase**2 + track_width**2)}"/>
-      <xacro:property name="wheel_Ixx" value="${(1/12) * wheel_mass * (3*wheel_radius**2 + wheel_width**2)}"/>
-      <xacro:property name="wheel_Iyy" value="${(1/12) * wheel_mass * (3*wheel_radius**2 + wheel_width**2)}"/>
-      <xacro:property name="wheel_Izz" value="${(1/2) * wheel_mass * wheel_radius**2}"/>
+    <model name='${prefix}caddy_ai2' canonical_link='${prefix}base_footprint'>
       <!-- ==================== ROBOT BASE ==================== -->
+      <!-- Base Footprint -->
+      <link name="${prefix}base_footprint">
+        <pose relative_to="__model__">0 0 0 0 0 0</pose>
+        <visual name="${prefix}base_footprint_visual">
+          <geometry>
+            <box>
+              <size>${vehicle_collision_length} ${vehicle_collision_width} 0.01</size>
+            </box>
+          </geometry>
+          <xacro:material_color rgba="${color_red}"/>
+        </visual>
+      </link>
+      <joint name="${prefix}base_joint" type="fixed">
+        <parent>${prefix}base_footprint</parent>
+        <child>${prefix}base_link</child>
+      </joint>
+      <!-- Base Link -->
       <link name='${prefix}base_link'>
-        <must_be_base_link>true</must_be_base_link>
+        <pose relative_to="${prefix}base_footprint">0 0 ${wheel_radius} 0 0 0</pose>
         <inertial>
           <mass>${mass}</mass>
@@ -59,22 +99,16 @@
           </geometry>
         </collision>
+        <sensor name="${prefix}navsat_sensor" type="navsat">
+          <always_on>1</always_on>
+          <update_rate>10</update_rate>
+          <pose>0 0 0 0 0 0</pose>
+          <xacro:if value="${namespace != ''}">
+            <topic>/${namespace}/navsat</topic>
+          </xacro:if>
+          <xacro:unless value="${namespace != ''}">
+            <topic>/navsat</topic>
+          </xacro:unless>
+        </sensor>
       </link>
-      <!-- Base Footprint -->
-      <link name="${prefix}base_footprint">
-        <pose relative_to="${prefix}base_link">${vehicle_collision_offset_x} 0.0 -${wheel_radius-0.01} 0 0 0</pose>
-        <visual name="${prefix}base_footprint_visual">
-          <geometry>
-            <box>
-              <size>${vehicle_collision_length} ${vehicle_collision_width} 0.01</size>
-            </box>
-          </geometry>
-          <xacro:material_color rgba="${color_red}"/>
-        </visual>
-      </link>
-      <joint name="${prefix}base_joint" type="fixed">
-        <parent>${prefix}base_link</parent>
-        <child>${prefix}base_footprint</child>
-        <pose relative_to='${prefix}base_footprint'/>
-      </joint>
       <!-- ==================== MACROS PARA RUEDAS ==================== -->
       <!-- Ruedas traseras: control de VELOCIDAD -->
@@ -254,12 +288,19 @@
       <plugin filename="gz_ros2_control-system"
               name="gz_ros2_control::GazeboSimROS2ControlPlugin">
-        <xacro:if value="${namespace != ''}">
-          <ros>
+        <ros>
+          <xacro:if value="${namespace != ''}">
             <namespace>/${namespace}</namespace>
-          </ros>
-        </xacro:if>
+          </xacro:if>
+          <remapping>bicycle_steering_controller/tf_odometry:=/tf</remapping>
+        </ros>
         <parameters>$(find caddy_ai2_ros2_gazebo_simulation)/bringup/config/controllers_simulation.yaml</parameters>
       </plugin>
     </model>
   </xacro:macro>
+  <!-- ============================================ -->
+  <!-- Auto-instantiate for standalone use          -->
+  <!-- ============================================ -->
+  <xacro:caddy_ai2_robot
+    prefix="$(arg prefix)"
+    namespace="$(arg namespace)"/>
 </sdf>

File: description/sdf/caddy_ai2_world.sdf.xacro (robot description, xacro)
@@ -4,25 +4,5 @@
   <!-- https://sdformat.org/spec/1.11/sdf/ -->
   <!-- ============================================ -->
-  <!-- 1. Definir argumentos globales               -->
-  <!-- ============================================ -->
-  <xacro:arg name="robot1_prefix" default="robot1_"/>
-  <xacro:arg name="robot1_x" default="0"/>
-  <xacro:arg name="robot1_y" default="0"/>
-  <xacro:arg name="robot1_yaw" default="0"/>
-  <xacro:arg name="robot2_prefix" default="robot2_"/>
-  <xacro:arg name="robot2_x" default="3"/>
-  <xacro:arg name="robot2_y" default="0"/>
-  <xacro:arg name="robot2_yaw" default="0"/>
-  <xacro:arg name="robot3_prefix" default="robot3_"/>
-  <xacro:arg name="robot3_x" default="-3"/>
-  <xacro:arg name="robot3_y" default="2"/>
-  <xacro:arg name="robot3_yaw" default="1.57"/>
-  <!-- ============================================ -->
-  <!-- 2. Incluir dependencias                      -->
-  <!-- ============================================ -->
-  <xacro:include filename="$(find caddy_ai2_ros2_gazebo_simulation)/description/sdf/materials.sdf.xacro"/>
-  <xacro:include filename="$(find caddy_ai2_ros2_gazebo_simulation)/description/sdf/caddy_ai2_model.sdf.xacro"/>
-  <!-- ============================================ -->
-  <!-- 3. Definir el mundo                          -->
+  <!-- Definir el mundo                          -->
   <!-- ============================================ -->
   <world name='base_world'>
@@ -36,4 +16,5 @@
     <plugin filename="gz-sim-scene-broadcaster-system" name="gz::sim::systems::SceneBroadcaster"/>
     <plugin filename="gz-sim-imu-system" name="gz::sim::systems::Imu"/>
+    <plugin filename="gz-sim-navsat-system" name="gz::sim::systems::NavSat"/>
     <plugin filename="gz-sim-sensors-system" name="gz::sim::systems::Sensors">
       <render_engine>ogre2</render_engine>

Commit message: IMU and LiDAR working

File: description/sdf/caddy_ai2_model.sdf.xacro (robot description, xacro)
@@ -50,4 +50,34 @@
   <!-- Include materials -->
   <xacro:include filename="$(find caddy_ai2_ros2_gazebo_simulation)/description/sdf/materials.sdf.xacro"/>
+  <!-- ============================================ -->
+  <!-- Sensors parameters                           -->
+  <!-- ============================================ -->
+  <!-- IMU offset from base_link -->
+  <xacro:property name="imu_offset_x" value="0.7"/>
+  <xacro:property name="imu_offset_y" value="0.0"/>
+  <xacro:property name="imu_offset_z" value="0.4"/>
+  <!-- IMU Covariance values (TODO: Characterize and update noise parameters) -->
+  <xacro:property name="imu_covariance_gyro" value="0.0"/>
+  <xacro:property name="imu_covariance_accel" value="0.0"/>
+  <!-- IMU Update rate -->
+  <xacro:property name="imu_update_rate" value="100"/>
+  <!-- LIDAR offset from base_link -->
+  <xacro:property name="lidar_offset_x" value="${wheelbase/2 + 0.125}"/>
+  <xacro:property name="lidar_offset_y" value="0.0"/>
+  <xacro:property name="lidar_offset_z" value="0.22"/>
+  <!-- LIDAR Update rate -->
+  <xacro:property name="lidar_update_rate" value="75"/>
+  <!-- LIDAR Noise (TODO: Characterize and update noise parameters) -->
+  <xacro:property name="lidar_noise_stddev" value="0.01"/>
+  <!-- GPS offset from base_link -->
+  <xacro:property name="gps_offset_x" value="${-wheelbase/2}"/>
+  <xacro:property name="gps_offset_y" value="0.0"/>
+  <xacro:property name="gps_offset_z" value="0.5"/>
+  <!-- GPS Update rate -->
+  <xacro:property name="gps_update_rate" value="10"/>
+  <!-- GPS Noise (TODO: Characterize and update noise parameters) -->
+  <xacro:property name="gps_horiz_stddev" value="0.1"/>
+  <xacro:property name="gps_vert_stddev" value="0.1"/>
+  <!-- ======== END OF SENSORS PARAMETERS ========= -->
   <!-- ============================================ -->
   <!-- MACRO PRINCIPAL DEL ROBOT                    -->
@@ -296,4 +326,109 @@
         <parameters>$(find caddy_ai2_ros2_gazebo_simulation)/bringup/config/controllers_simulation.yaml</parameters>
       </plugin>
+      <!-- ================================================================================================= -->
+      <!-- =                      SENSORS CONFIGURATION SECTION: IMU, LIDAR & GPS                          = -->
+      <!-- ================================================================================================= -->
+      <!-- Definimos enlace y unión para la IMU: -->
+      <!-- IMU Link -->
+      <link name="${prefix}imu_link">
+        <pose relative_to="${prefix}base_link">${imu_offset_x} ${imu_offset_y} ${imu_offset_z} 0 0 0</pose>
+        <visual name="${prefix}imu_visual">
+          <geometry>
+            <box>
+              <size>0.05 0.05 0.02</size>
+            </box>
+          </geometry>
+          <xacro:material_color rgba="${color_black}"/>
+        </visual>
+        <sensor name="${prefix}imu_sensor" type="imu">
+          <always_on>true</always_on>
+          <!-- IMU Sampling (and publishing) rate -->
+          <update_rate>${imu_update_rate}</update_rate>
+          <visualize>true</visualize>
+          <xacro:if value="${namespace != ''}">
+            <topic>/${namespace}/imu</topic>
+          </xacro:if>
+          <xacro:unless value="${namespace != ''}">
+            <topic>/imu</topic>
+          </xacro:unless>
+          <gz_frame_id>${prefix}imu_link</gz_frame_id>
+          <imu>
+            <angular_velocity>
+              <x><noise type="gaussian"><mean>0.0</mean><stddev>${imu_covariance_gyro}</stddev></noise></x>
+              <y><noise type="gaussian"><mean>0.0</mean><stddev>${imu_covariance_gyro}</stddev></noise></y>
+              <z><noise type="gaussian"><mean>0.0</mean><stddev>${imu_covariance_gyro}</stddev></noise></z>
+            </angular_velocity>
+            <linear_acceleration>
+              <x><noise type="gaussian"><mean>0.0</mean><stddev>${imu_covariance_accel}</stddev></noise></x>
+              <y><noise type="gaussian"><mean>0.0</mean><stddev>${imu_covariance_accel}</stddev></noise></y>
+              <z><noise type="gaussian"><mean>0.0</mean><stddev>${imu_covariance_accel}</stddev></noise></z>
+            </linear_acceleration>
+          </imu>
+        </sensor>
+      </link>
+      <!-- IMU Joint -->
+      <joint name="${prefix}imu_joint" type="fixed">
+        <parent>${prefix}base_link</parent>
+        <child>${prefix}imu_link</child>
+      </joint>
+      <!-- Definimos enlace y unión para el LIDAR: -->
+      <!-- LIDAR Link -->
+      <link name="${prefix}lidar_link">
+        <pose relative_to="${prefix}base_link">${lidar_offset_x} ${lidar_offset_y} ${lidar_offset_z} 0 0 0</pose>
+        <visual name="${prefix}lidar_visual">
+          <geometry>
+            <cylinder>
+              <radius>0.08</radius>
+              <length>0.15</length>
+            </cylinder>
+          </geometry>
+          <xacro:material_color rgba="${color_blue}"/>
+        </visual>
+        <collision name="${prefix}lidar_collision">
+          <geometry>
+            <cylinder>
+              <radius>0.08</radius>
+              <length>0.15</length>
+            </cylinder>
+          </geometry>
+        </collision>
+        <sensor name="${prefix}lidar_sensor" type="gpu_lidar">
+          <always_on>true</always_on>
+          <update_rate>${lidar_update_rate}</update_rate>
+          <visualize>true</visualize>
+          <xacro:if value="${namespace != ''}">
+            <topic>/${namespace}/scan</topic>
+          </xacro:if>
+          <xacro:unless value="${namespace != ''}">
+            <topic>/scan</topic>
+          </xacro:unless>
+          <gz_frame_id>${prefix}lidar_link</gz_frame_id>
+          <lidar>
+            <scan>
+              <horizontal>
+                <samples>181</samples>
+                <resolution>1</resolution>
+                <min_angle>-1.570796</min_angle>
+                <max_angle>1.570796</max_angle>
+              </horizontal>
+            </scan>
+            <range>
+              <min>0.10</min> <max>80.0</max> <resolution>0.01</resolution> </range>
+            <noise>
+              <type>gaussian</type>
+              <mean>0.0</mean>
+              <stddev>${lidar_noise_stddev}</stddev> </noise>
+          </lidar>
+        </sensor>
+      </link>
+      <!-- LIDAR Joint -->
+      <joint name="${prefix}lidar_joint" type="fixed">
+        <parent>${prefix}base_link</parent>
+        <child>${prefix}lidar_link</child>
+      </joint>
+      <!-- Definimos enlace y unión para el GPS (TODO: Merge con rama GPS) -->
+      <!-- ================================================================================================= -->
+      <!-- ============================== END OF SENSORS PLACEMENT SECTION ================================= -->
+      <!-- ================================================================================================= -->
     </model>
   </xacro:macro>

File: description/sdf/caddy_ai2_world.sdf.xacro (robot description, xacro)
@@ -104,4 +104,14 @@
     <!-- spawn_robot.launch.py, no en el world SDF.   -->
     <!-- ============================================ -->
+    <!-- ==================== 5. CONFIG PARA SIMULACIÓN DE SENSORES =========================== -->
+    <!-- GPS Plugin and coordinates transform configuration -->
+    <spherical_coordinates>
+      <surface_model>EARTH_WGS84</surface_model>
+      <world_frame_orientation>ENU</world_frame_orientation> <latitude_deg>40.4168</latitude_deg>
+      <longitude_deg>-3.7038</longitude_deg>
+      <elevation>600.0</elevation>
+      <heading_deg>0</heading_deg>
+    </spherical_coordinates>
+    <!-- ====================================================================================== -->
   </world>
 </sdf>
